File: kicad/mcu.sch (KiCad schematic (older format))
At the start: 9 parts, among them M1 M50-3130545, SW1 SW_Push, Y1 32.768 kHz

Commit message: switched the size of C14
Parts:
- C14: footprint Capacitor_SMD:C_0805_2012Metric -> Capacitor_SMD:C_0603_1608Metric
Changed lines of the file:
@@
 F 0 "C14" H 6615 3796 50  0000 L CNN
 F 1 "4.7 µF" H 6615 3705 50  0000 L CNN
-F 2 "Capacitor_SMD:C_0805_2012Metric" H 6538 3600 50  0001 C CNN
+F 2 "Capacitor_SMD:C_0603_1608Metric" H 6538 3600 50  0001 C CNN
 F 3 "~" H 6500 3750 50  0001 C CNN
 	1    6500 3750
